File: PCB/advance schematic/advance schematic.kicad_pcb (KiCad board)
At the start: 2 copper layers, 129.5 x 77.5 mm, 27 parts, among them J1 Conn_01x02_Pin, SW2 sw_pickup, SW3 sw_speed_down, SW4 sw_mode_sensor, SW5 switch, U1 ESP32-DEVKITC-32E, U2 GY-521

Commit message: 19/10/2026 10.07
Parts:
- removed REF** (x4): MountingHole_3mm, MountingHole:MountingHole_3mm
- added M3: MountingHole_3.2mm_M3, MountingHole:MountingHole_3.2mm_M3, F.Cu at (90.0, 130.0)
- added M3: MountingHole_3.2mm_M3, MountingHole:MountingHole_3.2mm_M3, F.Cu at (209.0, 63.5)
- added M3: MountingHole_3.2mm_M3, MountingHole:MountingHole_3.2mm_M3, F.Cu at (210.5, 130.0)
- added M3: MountingHole_3.2mm_M3, MountingHole:MountingHole_3.2mm_M3, F.Cu at (91.0, 62.5)
- renumbered JO2 to JO3, JO1 to JO4
Connections:
- net /+5V renamed +5V
- JO3 pad 3: /JOY.VRx1 -> /JOY.VRx2
- JO3 pad 4: /JOY.VRy1 -> /JOY.VRy2
- JO4 pad 3: /JOY.VRx2 -> /JOY.VRx1
- JO4 pad 4: /JOY.VRy2 -> /JOY.VRy1
Routing:
- net GND: track 226.2 -> 0.00 mm
- net /JOY.VRx1: track 32.4 -> 68.8 mm
- net /JOY.VRy1: track 35.6 -> 66.2 mm
- net /JOY.VRx2: track 66.6 -> 36.0 mm
- net /JOY.VRy2: track 61.1 -> 39.6 mm
- net Net-(R9-Pad1): track 106.3 -> 115.8 mm
- net +5V: track 145.2 -> 140.9 mm
- net /CONTROL.up: track 65.6 -> 62.3 mm, vias 1 -> 0
- net /19: track 50.4 -> 52.9 mm
- net Net-(TP1-OUT-): track 81.2 -> 79.8 mm
- net Net-(R6-Pad1): track 115.6 -> 116.9 mm, vias 0 -> 1
- net /<NO NET>: track 72.9 -> 74.0 mm
- net /SCL: track 42.2 -> 43.3 mm, vias 0 -> 1
- net /SDA: track 45.5 -> 44.6 mm
- net /CONTROL.drop: vias 1 -> 0
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- added copper zone on B.Cu, net GND
